Commit message: [Coding] Add transformation for nissan leaf

File: src/bringup/urdf/sensor_box.urdf.xacro (robot description, xacro)
@@ -1,5 +1,6 @@
 <?xml version="1.0"?>
-<robot xmlns:xacro="http://www.ros.org/wiki/xacro" name="sensor_box">
-    <link name="base_link" />
+<robot xmlns:xacro="http://www.ros.org/wiki/xacro">
+<xacro:macro name = "sensor_box" params = "parent *origin">
+    <link name="box_link" />
     <xacro:property name="config_file" value="$(find bringup)/param/tf_sensors_params.yaml" />
     <xacro:property name="geom" value="${xacro.load_yaml(config_file)['sensor_geometry']}" />
@@ -15,7 +16,11 @@
     <xacro:property name="f_roll" value="${math.radians(rg['front_roll_deg'])}" />
     <xacro:property name="r_roll" value="${math.radians(rg['rear_roll_deg'])}" />
+    <joint name="box_link_joint" type="fixed">
+        <parent link="${parent}"/>
+        <child link="box_link"/>
+        <xacro:insert_block name="origin" /> </joint>
     <link name="radar_front_left" />
     <joint name="base_to_radar_fl" type="fixed">
-        <parent link="base_link"/>
+        <parent link="box_link"/>
         <child link="radar_front_left"/>
         <origin xyz="${f_dist * math.cos(f_yaw_rad)} ${f_dist * math.sin(f_yaw_rad)} ${h}"
@@ -24,12 +29,12 @@
     <link name="radar_front_right" />
     <joint name="base_to_radar_fr" type="fixed">
-        <parent link="base_link"/>
+        <parent link="box_link"/>
         <child link="radar_front_right"/>
-        <origin xyz="${f_dist * math.cos(-f_yaw_rad)} ${f_dist * math.sin(-f_yaw_rad)} ${h}"
+                <origin xyz="${f_dist * math.cos(-f_yaw_rad)} ${f_dist * math.sin(-f_yaw_rad)} ${h}"
                 rpy="${f_roll} ${f_pitch} ${-f_yaw_rad}" />
     </joint>
     <link name="radar_rear_left" />
     <joint name="base_to_radar_rl" type="fixed">
-        <parent link="base_link"/>
+        <parent link="box_link"/>
         <child link="radar_rear_left"/>
         <origin xyz="${-r_dist * math.cos(r_yaw_rad)} ${r_dist * math.sin(r_yaw_rad)} ${h}"
@@ -38,5 +43,5 @@
     <link name="radar_rear_right" />
     <joint name="base_to_radar_rr" type="fixed">
-        <parent link="base_link"/>
+        <parent link="box_link"/>
         <child link="radar_rear_right"/>
         <origin xyz="${-r_dist * math.cos(-r_yaw_rad)} ${r_dist * math.sin(-r_yaw_rad)} ${h}"
@@ -48,13 +53,13 @@
     </xacro:zed_camera>
     <joint name="zed_front_mount_joint" type="fixed">
-        <parent link="base_link" />
+        <parent link="box_link" />
         <child link="zed_front_camera_link" />
         <origin xyz="${cg['front_distance']} 0.0 ${cg['height']}" rpy="0 0 0" />
     </joint>
     <xacro:zed_camera name="zed_rear" model="zedx">
-        <gnss_origin/>
+       <gnss_origin/>
     </xacro:zed_camera>
     <joint name="zed_rear_mount_joint" type="fixed">
-        <parent link="base_link" />
+        <parent link="box_link" />
         <child link="zed_rear_camera_link" />
         <origin xyz="${-cg['rear_distance']} 0.0 ${cg['height']}" rpy="0 0 ${math.pi}" />
@@ -64,5 +69,5 @@
     </xacro:zed_camera>
     <joint name="zed_left_mount_joint" type="fixed">
-        <parent link="base_link" />
+        <parent link="box_link" />
         <child link="zed_left_camera_link" />
         <origin xyz="0.0 ${cg['left_distance']} ${cg['height']}" rpy="0 0 ${math.pi/2}" />
@@ -72,7 +77,8 @@
     </xacro:zed_camera>
     <joint name="zed_right_mount_joint" type="fixed">
-        <parent link="base_link" />
+        <parent link="box_link" />
         <child link="zed_right_camera_link" />
         <origin xyz="0.0 ${-cg['right_distance']} ${cg['height']}" rpy="0 0 ${-math.pi/2}" />
     </joint>
+</xacro:macro>
 </robot>
